Commit message: Add my_folder to new-1 branch

File: robot_arm_pkg/urdf/slide_robot_arm.urdf (robot description, URDF)
Before this commit: robot sliding_arm, 8 links, 7 joints
Links:
- link link1: mass 0.5 -> 1.3; geometry collision cylinder length=0.2 radius=0.2; visual cylinder length=0.2 radius=0.2
- link link2: mass 0.3 -> 1; geometry collision cylinder length=0.2 radius=0.2; visual cylinder length=0.2 radius=0.2
- link rotating2_link: mass 0.4 -> 1.1; geometry collision cylinder length=0.4 radius=0.15; visual cylinder length=0.4 radius=0.15
- link rotating_link: mass 1 -> 1.6; geometry collision cylinder length=0.7 radius=0.2; visual cylinder length=0.7 radius=0.2
- link slider_link: mass 1.45 -> 1; geometry collision box size=0.5 0.5 0.15; visual box size=0.5 0.5 0.15
Joints:
- joint rotating_joint: limit lower=-1.40 upper=1.40 effort=1000.0 velocity=0.5 -> lower=-1.40 upper=1.40 effort=100.0 velocity=0.5
